Commit message: Update GEN3_URDF_V12.urdf

File: kortex_description/arms/gen3/7dof/urdf/GEN3_URDF_V12.urdf (robot description, URDF)
Before this commit: robot GEN3_URDF_V12, 9 links, 8 joints
Links:
- link Bracelet_Link: geometry collision mesh filename=package://kortex_description/arms/gen3/meshes/bracelet_Link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; visual mesh filename=package://kortex_description/arms/gen3/meshes/bracelet_Link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
- link ForeArm_Link: geometry collision mesh filename=package://kortex_description/arms/gen3/meshes/forearm_Link.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; visual mesh filename=package://kortex_description/arms/gen3/meshes/ForeArm_Link.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
- link HalfArm1_Link: geometry collision mesh filename=package://kortex_description/arms/gen3/meshes/halfarm1_Link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; visual mesh filename=package://kortex_description/arms/gen3/meshes/halfarm1_Link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
- link HalfArm2_Link: geometry collision mesh filename=package://kortex_description/arms/gen3/meshes/halfarm2_Link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; visual mesh filename=package://kortex_description/arms/gen3/meshes/halfarm2_Link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
- link Shoulder_Link: geometry collision mesh filename=package://kortex_description/arms/gen3/meshes/shoulder_link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; visual mesh filename=package://kortex_description/arms/gen3/meshes/Shoulder_Link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
- link SphericalWrist1_Link: geometry collision mesh filename=package://kortex_description/arms/gen3/meshes/sphericalwris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; visual mesh filename=package://kortex_description/arms/gen3/meshes/sphericalwris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
- link SphericalWrist2_Link: geometry collision mesh filename=package://kortex_description/arms/gen3/meshes/sphericalwris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; visual mesh filename=package://kortex_description/arms/gen3/meshes/sphericalwris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
